File: kicad_files/ds_lite_tv_out/ds_lite_tv_out.kicad_pcb (KiCad board)
At the start: 2 copper layers, 25.4 x 6.6 mm, 17 parts

Commit message: updated files
Other:
- board text added: "1"
- board text added: "2"
- board text added: "3"
- board text added: "4"
- board text removed: "6"
- board text removed: "7"
- board text removed: "8"
- board text removed: "9"
Changed lines of the file:
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@@
     (effects (font (size 1 1) (thickness 0.15)) (justify mirror))
   )
-  (gr_text "7" (at 130.36 79.42) (layer "B.SilkS")
+  (gr_text "3" (at 130.36 79.42) (layer "B.SilkS")
     (effects (font (size 1 1) (thickness 0.15)) (justify mirror))
   )
@@
     (effects (font (size 1 1) (thickness 0.15)) (justify mirror))
   )
-  (gr_text "5" (at 122.45 79.325) (layer "B.SilkS")
+  (gr_text "1" (at 122.45 79.325) (layer "B.SilkS")
     (effects (font (size 1 1) (thickness 0.15)) (justify mirror))
   )
-  (gr_text "8" (at 134.39 79.37) (layer "B.SilkS")
+  (gr_text "4" (at 134.39 79.37) (layer "B.SilkS")
     (effects (font (size 1 1) (thickness 0.15)) (justify mirror))
   )
@@
     (effects (font (size 1 1) (thickness 0.15)) (justify mirror))
   )
-  (gr_text "9" (at 138.19 79.37) (layer "B.SilkS")
+  (gr_text "5" (at 138.19 79.37) (layer "B.SilkS")
     (effects (font (size 1 1) (thickness 0.15)) (justify mirror))
   )
@@
     (effects (font (size 1 1) (thickness 0.15)) (justify mirror))
   )
-  (gr_text "6" (at 126.38 79.33) (layer "B.SilkS")
+  (gr_text "2" (at 126.38 79.33) (layer "B.SilkS")
     (effects (font (size 1 1) (thickness 0.15)) (justify mirror))
   )
